Commit message: (Longinus) Add the lance as an SDF file.

File: longinuslance_description/urdf/lance_longinus_mesh.urdf (robot description, URDF)
Before this commit: robot lance_longinus, 1 links, 0 joints
Links:
- link base_link: geometry visual mesh filename=/home/n130s/link/ROS/indigo_trusty/cws_spaceexploration/src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 scale=0.02 0.02 0.024
